File: Hardware/BC127_Breakout.brd (EAGLE design)
At the start: 63.5 x 33 mm, 38 parts, among them Q1 MOSFET-NCHANNELBSS138, Q2 MOSFET-NCHANNELBSS138, Q3 MMBT4403, U2 MIC5219 3.3V

Commit message: Changed TCream
-Changed TCream for more paste application to allow for better reflow to
the BC127 module
Parts:
- U1: value (none) -> BC127; device SparkFun-RF:BC127 -> SparkFun-RF:BC127_XTRA_PASTE
Changed lines of the file:
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@@
 <?xml version="1.0" encoding="utf-8"?>
 <!DOCTYPE eagle SYSTEM "eagle.dtd">
-<eagle version="6.5.0">
+<eagle version="6.4">
 <drawing>
 <settings>
@@
 <setting verticaltext="up"/>
 </settings>
-<grid distance="0.05" unitdist="inch" unit="inch" style="lines" multiple="1" display="yes" altdistance="0.01" altunitdist="inch" altunit="inch"/>
+<grid distance="0.05" unitdist="inch" unit="inch" style="lines" multiple="1" display="yes" altdistance="0.005" altunitdist="inch" altunit="inch"/>
 <layers>
 <layer number="1" name="Top" color="4" fill="1" visible="yes" active="yes"/>
@@
 <layer number="19" name="Unrouted" color="6" fill="1" visible="yes" active="yes"/>
 <layer number="20" name="Dimension" color="6" fill="1" visible="yes" active="yes"/>
-<layer number="21" name="tPlace" color="6" fill="1" visible="yes" active="yes"/>
-<layer number="22" name="bPlace" color="6" fill="1" visible="yes" active="yes"/>
+<layer number="21" name="tPlace" color="16" fill="1" visible="yes" active="yes"/>
+<layer number="22" name="bPlace" color="14" fill="1" visible="yes" active="yes"/>
 <layer number="23" name="tOrigins" color="15" fill="1" visible="yes" active="yes"/>
 <layer number="24" name="bOrigins" color="15" fill="1" visible="yes" active="yes"/>
@@
 </autorouter>
 <elements>
-<element name="U1" library="SparkFun-RF" package="BC127" value="" x="8.78" y="15.298" rot="R90"/>
+<element name="U1" library="SparkFun-RF" package="BC127_XTRA_PASTE" value="BC127" x="8.78" y="15.298" rot="R90"/>
 <element name="Q1" library="SparkFun-DiscreteSemi" package="SOT23" value="MOSFET-NCHANNELBSS138" x="39.37" y="8.89" rot="R180">
 <attribute name="PROD_ID" value="TRANS-00830" x="13.97" y="54.61" size="1.778" layer="27" rot="R180" display="off"/>
